File: board/nixie_clock.brd (EAGLE design)
At the start: 130 x 79 mm, 48 parts, among them U1 AMS1117-5.0, U2 SN74141N

Commit message: final board adjustments
Parts:
- moved U$2 2.83 mm to (6.00, 6.00)
Changed lines of the file:
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@@
 </element>
 <element name="U$1" library="holes" library_urn="urn:adsk.eagle:library:237" package="2,8" package3d_urn="urn:adsk.eagle:package:14271/1" value="" x="6" y="73" smashed="yes"/>
-<element name="U$2" library="holes" library_urn="urn:adsk.eagle:library:237" package="2,8" package3d_urn="urn:adsk.eagle:package:14271/1" value="" x="4" y="4" smashed="yes"/>
+<element name="U$2" library="holes" library_urn="urn:adsk.eagle:library:237" package="2,8" package3d_urn="urn:adsk.eagle:package:14271/1" value="" x="6" y="6" smashed="yes"/>
 <element name="U$3" library="holes" library_urn="urn:adsk.eagle:library:237" package="2,8" package3d_urn="urn:adsk.eagle:package:14271/1" value="" x="124" y="73" smashed="yes"/>
 <element name="U$4" library="holes" library_urn="urn:adsk.eagle:library:237" package="2,8" package3d_urn="urn:adsk.eagle:package:14271/1" value="" x="124" y="6" smashed="yes"/>

Commit message: PCB redesign
Parts:
- removed INPUT, SHNT: 22-23-2021, con-molex:22-23-2021
- removed OK1, OK2, OK3, OK4, OK5: SFH618A-5X007, optocoupler:SMD4-7
- removed R11, R6, R7, R8, R9: 22k, rcl:0204/7
- added 10H, 10MIN, 1H, 1MIN, DOT: PC-TLP127, we-opto:MINIFLAT4
- added 12V: TERMINAL_2P, KF301-2P-Terminal:KF301-2P
- added 12V_INPUT: DCJ0202, con-jack:DCJ0202
- 200V: value (none) -> TERMINAL_2P; device con-amp-quick:03P -> KF301-2P-Terminal:KF301-2P
- R10: value 670 -> 56k
- RTC: device con-lstb:MA03-1 -> con-lstb:MA05-1
- U$1, U$2, U$3, U$4: device holes:2,8 -> holes:3,2
- moved U$2 135.7 mm to (124.0, 73.0)
- moved U$4 118.0 mm to (6.00, 6.00)
- moved U$3 67.0 mm to (124.0, 6.00)
- moved 200V 42.2 mm to (6.00, 56.0), flipped to the top
- moved C9 34.9 mm to (105.1, 30.0)
- moved C10 27.1 mm to (96.6, 29.9)
- moved C5 25.1 mm to (113.0, 29.7)
- moved L3 21.5 mm to (48.8, 28.2)
- moved R5 18.2 mm to (109.3, 16.4)
- moved C3 17.7 mm to (55.6, 28.3)
- moved C8 17.5 mm to (69.1, 28.1)
- moved U1 17.2 mm to (77.0, 35.8)
- moved R4 16.4 mm to (65.5, 8.39)
- moved C7 15.5 mm to (67.3, 36.9)
- moved C1 15.3 mm to (62.0, 28.2)
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Connections:
- removed net N$1: D1.A, INPUT.1
- removed net N$21: ARDUINO_NANO1.24, BUTTONS.8, R1.2
- removed net N$22: ARDUINO_NANO1.10, RTC.2
- removed net N$23: ARDUINO_NANO1.11, RTC.1
- new net 5V: ARDUINO_NANO1.12
- new net N$3: ARDUINO_NANO1.26, RTC.1
- new net N$7: ARDUINO_NANO1.24, RTC.3
- net +12V: no longer SHNT.2
- net +5V: now also R1.2, R5.2, RTC.5; no longer ARDUINO_NANO1.12, R1.1, R11.1, R5.1, R6.1, R7.1, R8.1, R9.1
- net 12V: now also 12V.2, 12V_INPUT.1, D1.A; no longer 200V.2
- net 200V: now also 200V.2; no longer 200V.3
- net A_10H: now also 10H.4; no longer OK1.3
- net A_10MIN: now also 10MIN.4; no longer OK4.3
- net A_1H: now also 1H.4; no longer OK2.3
- net A_1MIN: now also 1MIN.4; no longer OK5.3
- net A_DOT: now also DOT.4; no longer OK3.3
- net GND: now also 12V.1, 12V_INPUT.2, 12V_INPUT.3, BUTTONS.2, RTC.4; no longer INPUT.2, SHNT.1
- net N$10: now also ARDUINO_NANO1.11, R1.1; no longer ARDUINO_NANO1.29, R9.2
- net N$15: now also 10H.1; no longer OK1.1
- net N$16: now also 10H.3, 10MIN.3, 1H.3, 1MIN.3, DOT.3; no longer OK1.2, OK2.2, OK3.2, OK4.2, OK5.2
- net N$17: now also ARDUINO_NANO1.9, BUTTONS.5; no longer ARDUINO_NANO1.28, BUTTONS.4, R8.2
- net N$18: now also ARDUINO_NANO1.29, BUTTONS.6; no longer ARDUINO_NANO1.27, BUTTONS.5, R7.2
- net N$19: now also ARDUINO_NANO1.28, BUTTONS.7; no longer ARDUINO_NANO1.26, BUTTONS.6, R6.2
- net N$20: now also ARDUINO_NANO1.27, BUTTONS.8; no longer ARDUINO_NANO1.25, BUTTONS.7, R5.2
- net N$26: now also 1H.1; no longer OK2.1
- net N$27: now also DOT.1; no longer OK3.1
- net N$28: now also 10MIN.1; no longer OK4.1
- net N$29: now also 1MIN.1; no longer OK5.1
- net N$4: now also ARDUINO_NANO1.25, RTC.2; no longer ARDUINO_NANO1.1, BUTTONS.2, R11.2
- net N$5: now also 10H.6, 10MIN.6, 1H.6, 1MIN.6, DOT.6; no longer OK1.4, OK2.4, OK3.4, OK4.4, OK5.4
- net N$9: now also ARDUINO_NANO1.10, BUTTONS.4, R5.1; no longer ARDUINO_NANO1.9, RTC.3
Routing:
- net N$26: track 138.1 -> 55.6 mm, vias 0 -> 2
- net N$7: track 0.00 -> 46.0 mm
- net 200V: track 30.8 -> 75.9 mm
- net K7: track 141.3 -> 179.4 mm, vias 4 -> 3
- net N$29: track 80.0 -> 43.9 mm
- net N$15: track 116.4 -> 84.0 mm, vias 1 -> 0
- net N$13: track 27.7 -> 59.1 mm
- net K0: track 179.6 -> 149.3 mm, vias 1 -> 2
- net K5: track 128.0 -> 157.3 mm, vias 2 -> 5
- net N$28: track 57.3 -> 29.5 mm, vias 1 -> 2
- net N$16: track 146.6 -> 125.3 mm, vias 3 -> 2
- net N$14: track 58.3 -> 37.3 mm
- net N$3: track 0.00 -> 20.7 mm
- net K4: track 146.9 -> 126.8 mm
- net N$22: track 19.9 -> 0.00 mm
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Other:
- board text added: "+"
- board text added: "-"
- board text added: "200V"
- board text added: "b1"
- board text added: "e"
- board text added: "github.com/peternagy96/nixie_clock"
- board text added: "gnd"
- board text added: "s1d"
- board text added: "s1u"
- board text added: "s2d"
- board text added: "s2u"
- board text removed: "Nixie Clock"
